File: KiCad_Traffic_Light_Controller_guide/KiCad_JLPCB_template_2layers/Traffic_Light_Controller/Traffic_Light_Controller.kicad_pcb (KiCad board)
At the start: 2 copper layers, 124.2 x 91.4 mm, 65 parts, among them J1 Conn_02x08_Odd_Even, J2 Conn_02x08_Odd_Even, J3 Conn_02x05_Odd_Even, J4 +5V, SW1 RST, SW2 OVRRIDE, SW3 EN, U1 SM420561N, U2 SM420561N, U3 LM1117DT-3.3

Commit message: update
Other:
- board text added: "Cid Lawrenc C. Regalado 22 April 2026 Computer Engineering Technology Department Technological University of the Philippines-Visayas"
- board text removed: "Cid Lawrenc C. Regalado 19 April 2026 Computer Engineering Technology Department Technological University of the Philippines-Visayas"

Commit message: KICAD 9
Parts:
- removed G***: LOGO, LOGO
- moved C4 18.5 mm to (117.5, 81.5)
- moved D10 18.5 mm to (105.7, 128.8)
- moved D11 18.5 mm to (189.9, 116.4)
- moved D13 18.5 mm to (173.0, 116.1)
- moved D2 18.5 mm to (172.1, 74.6)
- moved D4 18.5 mm to (135.6, 110.6)
- moved D5 18.5 mm to (135.6, 121.2)
- moved D6 18.5 mm to (135.6, 131.8)
- moved D7 18.5 mm to (204.5, 69.2)
- moved H2 18.5 mm to (214.8, 56.8)
- moved H4 18.5 mm to (96.8, 141.9)
- moved J1 18.5 mm to (129.4, 77.3)
- moved J3 18.5 mm to (136.9, 64.8)
- moved J4 18.5 mm to (107.3, 65.1)
- moved R1 18.5 mm to (190.3, 61.3)
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Routing:
- net /NS_HEX_A: track 106.3 -> 107.8 mm
- net /EN: track 146.5 -> 147.8 mm
Other:
- board size 124.2 x 91.4 mm -> 124.2 x 91.3 mm
- board text added: "Regalado, Cid Lawrenc C. 22 April 2026 Computer Engineering Technology Department Technological University of the Philippines Visayas"
- board text removed: "Cid Lawrenc C. Regalado 22 April 2026 Computer Engineering Technology Department Technological University of the Philippines-Visayas"

Commit message: update
Parts:
- added G***: LOGO, LOGO, F.Cu at (201.5, 135.0)
